File: ESP32_Environmental_IMU_Board/Hardware/Environmental_sensor_MPU6050/Environmental_sensor_MPU6050.kicad_pcb (KiCad board)
At the start: 4 copper layers, 72.9 x 62.9 mm, 86 parts, among them IC1 MP1584EN-LF-Z, J1 USB_C_Receptacle_USB2.0_16P, J2 Conn_01x02, J3 Conn_01x04_Pin, J4 Conn_01x04_Pin, J5 Micro_SD_Card, SW1 SW_Push, SW2 SW_Push, U1 MCP73831-2-OT, U10 MLX90614ESF-BAA-000-TU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

Commit message: PCB Layout done
Parts:
- removed D5: D, Diode_SMD:D_SOD-123F
- removed R10: 0, Resistor_SMD:R_0603_1608Metric
- added H1: MountingHole_Pad, MountingHole:MountingHole_2.2mm_M2_Pad_Via, F.Cu at (71.0, 51.9)
- added H2: MountingHole_Pad, MountingHole:MountingHole_2.2mm_M2_Pad_Via, F.Cu at (138.1, 51.9)
- added H3: MountingHole_Pad, MountingHole:MountingHole_2.2mm_M2_Pad_Via, F.Cu at (70.9, 103.2)
- added H4: MountingHole_Pad, MountingHole:MountingHole_2.2mm_M2_Pad_Via, F.Cu at (138.1, 103.1)
- moved U7 21.9 mm to (106.6, 83.3)
- moved C23 15.0 mm to (109.1, 103.4), turned to -90 degrees
- moved R_LED2 14.0 mm to (95.3, 61.2)
- moved D6 13.0 mm to (98.6, 61.2)
- moved U9 10.7 mm to (106.7, 103.4)
- moved D3 7.16 mm to (85.4, 83.0), turned to 0 degrees
- moved C13 5.89 mm to (95.8, 80.5), turned to 0 degrees
- moved R8 5.50 mm to (89.9, 82.2)
- moved R9 5.43 mm to (92.3, 81.2)
- moved TP1 4.77 mm to (89.8, 51.2), turned to 0 degrees
- moved U10 3.62 mm to (107.1, 94.9)
- moved C24 3.62 mm to (112.5, 98.9)
- moved C25 3.62 mm to (113.4, 96.2)
- moved TP2 3.19 mm to (85.8, 51.2), turned to -90 degrees
- moved BT1 2.91 mm to (120.8, 84.4)
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Connections:
- C10 pad 1: 3V3 -> ESP32_3V3
- C11 pad 1: 3V3 -> ESP32_3V3
- C14 pad 1: 3V3 -> ESP32_3V3
- C15 pad 1: 3V3 -> ESP32_3V3
- TP2 pad 1: Net-(D5-A) -> ESP32_3V3
- U2 pad 5: 3V3 -> ESP32_3V3
Routing:
- net GND: track 0.00 -> 140.1 mm, vias 0 -> 70
- net SDA/IO8: track 0.00 -> 122.1 mm, vias 0 -> 8
- net SCL/IO9: track 0.00 -> 117.8 mm, vias 0 -> 4
- net BOOT: track 0.00 -> 63.3 mm, vias 0 -> 2
- net ESP32_3V3: track 0.00 -> 63.0 mm, vias 0 -> 24
- net SCK: track 0.00 -> 61.7 mm, vias 0 -> 2
- net MOSI: track 0.00 -> 56.6 mm, vias 0 -> 4
- net CS: track 0.00 -> 55.3 mm, vias 0 -> 4
- net MISO: track 0.00 -> 51.8 mm, vias 0 -> 2
- net VBUS: track 0.00 -> 43.1 mm
- net CHIP-PU/RST/EN: track 0.00 -> 41.1 mm
- net Net-(D3-K): track 0.00 -> 33.4 mm, vias 0 -> 2
- net USB_D-: track 0.00 -> 30.0 mm
- net USB_D+: track 0.00 -> 29.7 mm
- net BAT+: track 0.00 -> 23.4 mm, vias 0 -> 2
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- added copper zone on F.Cu, net BAT+
- added copper zone on In2.Cu, net ESP32_3V3
- added copper zone on In1.Cu, net GND
Other:
- outline, holes or cut-outs redrawn
- board text added: "Indoor Environmental"
- board text added: "Quality (IEQ) Monitor"
- board text added: "RTC"
