File: ESP32_Environmental_IMU_Board/Hardware/Environmental_sensor_MPU6050/Environmental_sensor_MPU6050.kicad_pcb (KiCad board)
At the start: 4 copper layers, 72.9 x 62.9 mm, 88 parts, among them IC1 MP1584EN-LF-Z, J1 USB_C_Receptacle_USB2.0_16P, J2 Conn_01x02, J3 Conn_01x04_Pin, J4 Conn_01x04_Pin, J5 Micro_SD_Card, SW1 SW_Push, SW2 SW_Push, U1 MCP73831-2-OT, U10 MLX90614ESF-BAA-000-TU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

Commit message: Stitching vias added
Routing:
- net GND: vias 70 -> 137
