File: ESP32_Environmental_IMU_Board/Hardware/Environmental_sensor_MPU6050/Environmental_sensor_MPU6050.kicad_sch (KiCad schematic)
At the start: 86 parts, among them IC1 MP1584EN-LF-Z, J1 USB_C_Receptacle_USB2.0_16P, J2 Conn_01x02, J3 Conn_01x04_Pin, J4 Conn_01x04_Pin, J5 Micro_SD_Card, SW1 SW_Push, SW2 SW_Push, U1 MCP73831-2-OT, U10 MLX90614ESF-BAA-000-TU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

Commit message: PCB Layout done
Parts:
- removed D5: D, Diode_SMD:D_SOD-123F, symbol Device:D
- removed R10: 0, Resistor_SMD:R_0603_1608Metric, symbol Device:R
- added H1, H2, H3, H4: MountingHole_Pad, MountingHole:MountingHole_2.2mm_M2_Pad_Via, symbol Mechanical:MountingHole_Pad
Connections:
- net 3V3 is gone; now on net ESP32_3V3: C10.1, C11.1, C14.1, C15.1, U2.5 (VOUT)
- net ESP32_3V3: now also TP2.1
- net GND: now also H1.1, H2.1, H3.1, H4.1
Other:
- note added: "MOUNTING HOLES"
- moved on the sheet: C14, C15, TP1, TP2
