File: USB-C_Power_Supply/USB-C_Power_Supply/USB-C_Power_Supply.kicad_sch (KiCad schematic)
At the start: 41 parts, among them J1 USB_C_Receptacle_USB2.0_16P, J2 Screw_Terminal_01x02, J3 Conn_01x03_Pin, Q1 2N7002, SW1 SW_DIP_x03, U1 TPS70933DBVR, U2 USBLC6-2P6, U3 CH224A, U4 MC14051BDR2G

Commit message: ERC done!
Parts:
- removed C1, C4: 1uF, CL10B105KB8NQNC:CAPC1608X95N, symbol CL10B105KB8NQNC:CL10B105KB8NQNC
- removed C2, C5, C6: 0.1uF, CL05B104KB54PNC:CAPC1005X55N, symbol CL05B104KB54PNC:CL05B104KB54PNC
- added C1, C4: 1uF, symbol Device:C
- added C2, C5, C6: 0.1uF, symbol Device:C
Connections:
- net +3.3V: now also C6.1
- net +V_USB: now also C1.1, C2.1, C4.1, C5.1
- net GND: now also C1.2, C2.2, C4.2, C5.2, C6.2

Commit message: Schematic updated
Parts:
- removed C1: 1uF, symbol Device:C
- removed C3: 2.2uF, symbol Device:C
- removed R1: 10k, Resistor_SMD:R_0603_1608Metric, symbol Device:R
- removed U1: TPS70933DBVR, TPS70933DBVR:SOT95P280X145-5N, symbol TPS70933DBVR:TPS70933DBVR
- added C10: 1uF, symbol Device:C
- added C11: 0.1uF, symbol Device:C
- added C12, C16: 100nF, symbol Device:C
- added C13: 20pF, symbol Device:C
- added C14, C15, C7: 10uF, symbol Device:C
- added C8: 22uF, symbol Device:C
- added C9: 1nF, symbol Device:C
- added D10: 1N4148, Diode_THT:D_DO-35_SOD27_P7.62mm_Horizontal, symbol Diode:1N4148
- added D7: D_Zener, symbol Device:D_Zener
- added D8: D_TVS, symbol Device:D_TVS
- added D9: SS310, Diode_SMD:D_SMA, symbol Diode:SS310
- added L1: 15uH, symbol Device:L
- added Q2: PMOS, symbol Simulation_SPICE:PMOS
- added R17: 100k, Resistor_SMD:R_0603_1608Metric, symbol Device:R
- added R18: 1M, Resistor_SMD:R_0603_1608Metric, symbol Device:R
- added R19, R20: 22R, Resistor_SMD:R_0603_1608Metric, symbol Device:R
- added R21: 31.6k, Resistor_SMD:R_0603_1608Metric, symbol Device:R
- added R22: 10k, Resistor_SMD:R_0603_1608Metric, symbol Device:R
- added U5: MCP16331x-xCH, Package_TO_SOT_SMD:SOT-23-6, symbol Regulator_Switching:MCP16331x-xCH
- C2: value 0.1uF -> 10uF
- C4: value 1uF -> 10uF
Connections:
- net +3.3V: now also C13.1, C14.1, C15.1, D10.2 (A), L1.2, R21.2
- net +V_USB: now also C2.2, C4.2, C5.2, C6.2, D2.1 (K), D3.1 (K), D4.1 (K), D5.1 (K), D6.1 (K), H1.1, H2.1, H3.1, H4.1, J1.A1 (GND), J1.A12 (GND), J1.B1 (GND), J1.B12 (GND), J2.2 (Pin_2), J3.2 (Pin_2), Q1.2 (S), R5.2, R9.2, SW1.4, SW1.5, SW1.6, U2.2 (GND), U3.11 (GND), U4.7 (VEE), U4.8 (VSS), C10.1, C10.2, C11.1, C11.2, C14.2, C15.2, C16.1, C16.2, C7.1, C7.2, C8.1, C8.2, C9.2, D7.1 (K), D8.1 (A1), D9.2 (A), Q2.3 (S), R17.1, R18.1, R22.1, U5.2 (GND), U5.4 (EN), U5.5 (V_{IN}); no longer J1.A4 (VBUS), J1.A9 (VBUS), J1.B4 (VBUS), J1.B9 (VBUS)
- net CC1: now also R19.1; no longer J1.A5 (CC1)
- net CC2: now also R20.1; no longer J1.B5 (CC2)
- removed net GND: C2.2, C4.2, C5.2, C6.2, D2.1 (K), D3.1 (K), D4.1 (K), D5.1 (K), D6.1 (K), H1.1, H2.1, H3.1, H4.1, J1.A1 (GND), J1.A12 (GND), J1.B1 (GND), J1.B12 (GND), J1.SH (SHIELD), J2.2 (Pin_2), J3.2 (Pin_2), Q1.2 (S), R5.2, R9.2, SW1.4, SW1.5, SW1.6, U2.2 (GND), U3.11 (GND), U4.7 (VEE), U4.8 (VSS)
- new net: J1.A5 (CC1), R19.2
- new net: D8.2 (A2), J1.A4 (VBUS), J1.A9 (VBUS), J1.B4 (VBUS), J1.B9 (VBUS), Q2.1 (D)
- new net: J1.B5 (CC2), R20.2
- new net: C13.2, R21.1, R22.2, U5.3 (V_{FB})
- new net: C9.1, J1.SH (SHIELD), R18.2
- new net: C12.1, D10.1 (K), U5.1 (BOOST)
- new net: C12.2, D9.1 (K), L1.1, U5.6 (SW)
- new net: D7.2 (A), Q2.2 (G), R17.2
Other:
- moved on the sheet: C4, C5, C6, D1, D2, D3, D4, D5, D6, H1, H2, H3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
